File: heatedGripv2/heatedGripv2.kicad_sch (KiCad schematic)
At the start: 21 parts, among them J1 USB_C_Receptacle_USB2.0, J2 HEAT, J3 BATT, Q1 DMN3300U, SW1 SW_Push, U1 ATtiny204-SS, U2 MCP73811T-420I-OT, U3 REG710NA-3.3/3K

Commit message: Updated
Added extra ports and reviewed
Parts:
- removed J1: USB_C_Receptacle_USB2.0, Connector_USB:USB_C_Receptacle_GCT_USB4135-GF-A_6P_TopMnt_Horizontal, symbol Connector:USB_C_Receptacle_USB2.0
- added J1: TEMP, Connector_PinHeader_2.54mm:PinHeader_1x03_P2.54mm_Vertical, symbol Connector_Generic:Conn_01x03
- added J4: USB_C_Receptacle_PowerOnly_6P, Connector_USB:USB_C_Receptacle_GCT_USB4135-GF-A_6P_TopMnt_Horizontal, symbol Connector:USB_C_Receptacle_PowerOnly_6P
- added J5: PROG, Connector_PinHeader_2.54mm:PinHeader_1x03_P2.54mm_Vertical, symbol Connector_Generic:Conn_01x03
- D1: value LED -> QBL8RGB60D0-2897
Connections:
- net +3.3V: now also J1.2 (Pin_2), J5.2 (Pin_2)
- net +BATT: now also U3.3 (ENABLE)
- net GND: now also J1.3 (Pin_3), J4.A12 (GND), J4.B12 (GND), J4.S1 (SHIELD), J5.3 (Pin_3)
- net TEMP: now also U1.5 (PA7), J1.1 (Pin_1); no longer U1.10 (~{RESET}/PA0)
- net VBUS: now also J4.A9 (VBUS), J4.B9 (VBUS)
- net at R1.1: now also J4.A5 (CC1)
- net at R2.1: now also J4.B5 (CC2)
- new net PROG: J5.1 (Pin_1), U1.10 (~{RESET}/PA0)
- no-connect marks 11 -> 4
Other:
- moved on the sheet: C4, C5, C6, D1, R1, R2, SW1, U2

Commit message: Added Prod
Parts:
- C6: footprint Capacitor_SMD:C_0402_1005Metric_Pad0.74x0.62mm_HandSolder -> Capacitor_SMD:C_0603_1608Metric_Pad1.08x0.95mm_HandSolder
- Q1: value DMN3300U -> DMN2024U-7
Changed lines of the file:
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@@
       (effects (font (size 1.27 1.27)) (justify right))
     )
-    (property "Footprint" "Capacitor_SMD:C_0402_1005Metric_Pad0.74x0.62mm_HandSolder" (at 43.4848 157.48 0)
+    (property "Footprint" "Capacitor_SMD:C_0603_1608Metric_Pad1.08x0.95mm_HandSolder" (at 43.4848 157.48 0)
       (effects (font (size 1.27 1.27)) hide)
     )
@@
       (effects (font (size 1.27 1.27)) (justify left))
     )
-    (property "Value" "DMN3300U" (at 242.57 95.25 0)
+    (property "Value" "DMN2024U-7" (at 242.57 95.25 0)
       (effects (font (size 1.27 1.27)) (justify left))
     )
