File: heatedGripv2/heatedGripv2.kicad_pcb (KiCad board)
At the start: 2 copper layers, 25.4 x 16.5 mm, 21 parts, among them J1 USB_C_Receptacle_USB2.0, J2 HEAT, J3 BATT, Q1 DMN3300U, SW1 SW_Push, U1 ATtiny204-SS, U2 MCP73811T-420I-OT, U3 REG710NA-3.3/3K

Commit message: Updated
Added extra ports and reviewed
Parts:
- added J4: USB_C_Receptacle_PowerOnly_6P, Connector_USB:USB_C_Receptacle_GCT_USB4135-GF-A_6P_TopMnt_Horizontal, F.Cu at (121.3, 96.0)
- added J5: PROG, Connector_PinHeader_2.54mm:PinHeader_1x03_P2.54mm_Vertical, F.Cu at (134.1, 102.4)
- D1: value LED -> QBL8RGB60D0-2897
- J1: value USB_C_Receptacle_USB2.0 -> TEMP; footprint Connector_USB:USB_C_Receptacle_GCT_USB4135-GF-A_6P_TopMnt_Horizontal -> Connector_PinHeader_2.54mm:PinHeader_1x03_P2.54mm_Vertical
- moved J1 22.8 mm to (143.0, 102.4), turned to 90 degrees
- moved J2 5.08 mm to (145.7, 89.7)
- moved J3 5.02 mm to (145.7, 96.0)
Connections:
- R1 pad 1: Net-(J1-CC1) -> Net-(J4-CC1)
- R2 pad 1: Net-(J1-CC2) -> Net-(J4-CC2)
- U1 pad 10: /TEMP -> /PROG
- U1 pad 5: unconnected-(U1-PA7-Pad5) -> /TEMP
- U3 pad 3: unconnected-(U3-ENABLE-Pad3) -> +BATT
Routing:
- net +3.3V: track 7.24 -> 30.1 mm
- net /TEMP: track 0.00 -> 16.0 mm
- net GND: track 90.2 -> 102.8 mm
- net VBUS: track 14.4 -> 25.1 mm
- net /GATE: track 18.9 -> 9.75 mm
- net /PROG: track 0.00 -> 7.05 mm
- net /BAT_VOLT: track 12.7 -> 18.4 mm
- net Net-(J2-Pin_2): track 7.83 -> 13.2 mm
- net +BATT: track 43.3 -> 47.0 mm, vias 1 -> 2
- net Net-(J1-CC1): track 2.71 -> 0.00 mm
- net Net-(J4-CC1): track 0.00 -> 2.63 mm
- net Net-(J1-CC2): track 2.36 -> 0.00 mm
- net Net-(J4-CC2): track 0.00 -> 2.24 mm
Other:
- board size 25.4 x 16.5 mm -> 32.3 x 16.5 mm

Commit message: Added Prod
Parts:
- C6: footprint Capacitor_SMD:C_0402_1005Metric_Pad0.74x0.62mm_HandSolder -> Capacitor_SMD:C_0603_1608Metric_Pad1.08x0.95mm_HandSolder
- moved C6 0.51 mm to (137.9, 98.3)
Routing:
- net GND: track 102.8 -> 103.7 mm
Changed lines of the file:
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@@
     )
   )
-  (footprint "Capacitor_SMD:C_0402_1005Metric_Pad0.74x0.62mm_HandSolder" (layer "F.Cu")
-    (at 137.414 98.298 180)
-    (descr "Capacitor SMD 0402 (1005 Metric), square (rectangular) end terminal, IPC_7351 nominal with elongated pad for handsoldering. (Body size source: IPC-SM-782 page 76, https://www.pcb-3d.com/wordpress/wp-content/uploads/ipc-sm-782a_amendment_1_and_2.pdf), generated with kicad-footprint-generator")
+  (footprint "Capacitor_SMD:C_0603_1608Metric_Pad1.08x0.95mm_HandSolder" (layer "F.Cu")
+    (at 137.922 98.298 180)
+    (descr "Capacitor SMD 0603 (1608 Metric), square (rectangular) end terminal, IPC_7351 nominal with elongated pad for handsoldering. (Body size source: IPC-SM-782 page 76, https://www.pcb-3d.com/wordpress/wp-content/uploads/ipc-sm-782a_amendment_1_and_2.pdf), generated with kicad-footprint-generator")
     (tags "capacitor handsolder")
     (property "Sheetfile" "heatedGripv2.kicad_sch")
@@
     (property "ki_keywords" "cap capacitor")
     (attr smd)
-    (fp_text reference "C6" (at 0 -1.16) (layer "F.SilkS")
-        (effects (font (size 1 1) (thickness 0.15)))
-    )
-    (fp_text value "10n" (at 0 1.16) (layer "F.Fab")
-        (effects (font (size 1 1) (thickness 0.15)))
-    )
-    (fp_text user "${REFERENCE}" (at 0 0) (layer "F.Fab")
-        (effects (font (size 0.25 0.25) (thickness 0.04)))
-    )
-    (fp_line (start -0.115835 -0.36) (end 0.115835 -0.36)
-      (stroke (width 0.12) (type solid)) (layer "F.SilkS"))
-    (fp_line (start -0.115835 0.36) (end 0.115835 0.36)
-      (stroke (width 0.12) (type solid)) (layer "F.SilkS"))
-    (fp_line (start -1.08 -0.46) (end 1.08 -0.46)
-      (stroke (width 0.05) (type solid)) (layer "F.CrtYd"))
-    (fp_line (start -1.08 0.46) (end -1.08 -0.46)
-      (stroke (width 0.05) (type solid)) (layer "F.CrtYd"))
-    (fp_line (start 1.08 -0.46) (end 1.08 0.46)
-      (stroke (width 0.05) (type solid)) (layer "F.CrtYd"))
-    (fp_line (start 1.08 0.46) (end -1.08 0.46)
-      (stroke (width 0.05) (type solid)) (layer "F.CrtYd"))
-    (fp_line (start -0.5 -0.25) (end 0.5 -0.25)
-      (stroke (width 0.1) (type solid)) (layer "F.Fab"))
-    (fp_line (start -0.5 0.25) (end -0.5 -0.25)
-      (stroke (width 0.1) (type solid)) (layer "F.Fab"))
-    (fp_line (start 0.5 -0.25) (end 0.5 0.25)
-      (stroke (width 0.1) (type solid)) (layer "F.Fab"))
-    (fp_line (start 0.5 0.25) (end -0.5 0.25)
-      (stroke (width 0.1) (type solid)) (layer "F.Fab"))
-    (pad "1" smd roundrect (at -0.5675 0 180) (size 0.735 0.62) (layers "F.Cu" "F.Paste" "F.Mask") (roundrect_rratio 0.25)
+    (fp_text reference "C6" (at 0 -1.43 180) (layer "F.SilkS")
+        (effects (font (size 1 1) (thickness 0.15)))
+    )
+    (fp_text value "10n" (at 0 1.43 180) (layer "F.Fab")
+        (effects (font (size 1 1) (thickness 0.15)))
+    )
+    (fp_text user "${REFERENCE}" (at 0 0 180) (layer "F.Fab")
+        (effects (font (size 0.4 0.4) (thickness 0.06)))
+    )
+    (fp_line (start -0.146267 -0.51) (end 0.146267 -0.51)
+      (stroke (width 0.12) (type solid)) (layer "F.SilkS"))
+    (fp_line (start -0.146267 0.51) (end 0.146267 0.51)
+      (stroke (width 0.12) (type solid)) (layer "F.SilkS"))
+    (fp_line (start -1.65 -0.73) (end 1.65 -0.73)
+      (stroke (width 0.05) (type solid)) (layer "F.CrtYd"))
+    (fp_line (start -1.65 0.73) (end -1.65 -0.73)
+      (stroke (width 0.05) (type solid)) (layer "F.CrtYd"))
+    (fp_line (start 1.65 -0.73) (end 1.65 0.73)
+      (stroke (width 0.05) (type solid)) (layer "F.CrtYd"))
+    (fp_line (start 1.65 0.73) (end -1.65 0.73)
+      (stroke (width 0.05) (type solid)) (layer "F.CrtYd"))
+    (fp_line (start -0.8 -0.4) (end 0.8 -0.4)
+      (stroke (width 0.1) (type solid)) (layer "F.Fab"))
+    (fp_line (start -0.8 0.4) (end -0.8 -0.4)
+      (stroke (width 0.1) (type solid)) (layer "F.Fab"))
+    (fp_line (start 0.8 -0.4) (end 0.8 0.4)
+      (stroke (width 0.1) (type solid)) (layer "F.Fab"))
+    (fp_line (start 0.8 0.4) (end -0.8 0.4)
+      (stroke (width 0.1) (type solid)) (layer "F.Fab"))
+    (pad "1" smd roundrect (at -0.8625 0 180) (size 1.075 0.95) (layers "F.Cu" "F.Paste" "F.Mask") (roundrect_rratio 0.25)
       (net 2 "GND") (pintype "passive"))
-    (pad "2" smd roundrect (at 0.5675 0 180) (size 0.735 0.62) (layers "F.Cu" "F.Paste" "F.Mask") (roundrect_rratio 0.25)
+    (pad "2" smd roundrect (at 0.8625 0 180) (size 1.075 0.95) (layers "F.Cu" "F.Paste" "F.Mask") (roundrect_rratio 0.25)
       (net 13 "/BUTTON") (pintype "passive"))
-    (model "${KICAD6_3DMODEL_DIR}/Capacitor_SMD.3dshapes/C_0402_1005Metric.wrl"
+    (model "${KICAD6_3DMODEL_DIR}/Capacitor_SMD.3dshapes/C_0603_1608Metric.wrl"
       (offset (xyz 0 0 0))
       (scale (xyz 1 1 1))
@@
   (segment (start 130.556 93.3185) (end 129.082 93.3185) (width 0.25) (layer "F.Cu") (net 2))
   (segment (start 126.1259 100.198) (end 125.2319 101.092) (width 0.25) (layer "F.Cu") (net 2))
+  (segment (start 138.7845 97.696) (end 138.684 97.5955) (width 0.25) (layer "F.Cu") (net 2))
   (segment (start 120.65 92.0689) (end 120.65 92.116) (width 0.25) (layer "F.Cu") (net 2))
   (segment (start 130.556 92.9627) (end 130.556 93.3185) (width 0.25) (layer "F.Cu") (net 2))
   (segment (start 120.65 90.842) (end 120.65 92.0689) (width 0.25) (layer "F.Cu") (net 2))
+  (segment (start 138.7845 98.298) (end 138.7845 97.696) (width 0.25) (layer "F.Cu") (net 2))
   (segment (start 128.775 96.6205) (end 128.1665 96.012) (width 0.25) (layer "F.Cu") (net 2))
   (segment (start 139.192 102.362) (end 139.192 101.1851) (width 0.25) (layer "F.Cu") (net 2))
-  (segment (start 137.9815 93.574) (end 136.3555 91.948) (width 0.25) (layer "F.Cu") (net 2))
-  (segment (start 137.9815 98.298) (end 137.9815 93.574) (width 0.25) (layer "F.Cu") (net 2))
+  (segment (start 137.6249 99.0861) (end 138.413 98.298) (width 0.25) (layer "F.Cu") (net 2))
   (segment (start 139.192 100.6533) (end 137.6249 99.0861) (width 0.25) (layer "F.Cu") (net 2))
   (segment (start 128.2388 91.44) (end 128.6455 91.44) (width 0.25) (layer "F.Cu") (net 2))
@@
   (segment (start 128.1665 94.234) (end 127.1495 93.217) (width 0.25) (layer "F.Cu") (net 2))
   (segment (start 126.1259 100.198) (end 125.2119 99.284) (width 0.25) (layer "F.Cu") (net 2))
+  (segment (start 138.684 94.2765) (end 136.3555 91.948) (width 0.25) (layer "F.Cu") (net 2))
   (segment (start 128.6951 88.8294) (end 128.6245 88.9) (width 0.25) (layer "F.Cu") (net 2))
-  (segment (start 137.6249 99.0861) (end 137.9815 98.7295) (width 0.25) (layer "F.Cu") (net 2))
   (segment (start 129.082 93.3185) (end 128.1665 94.234) (width 0.25) (layer "F.Cu") (net 2))
   (segment (start 123.9029 92.0689) (end 124.23 92.0689) (width 0.25) (layer "F.Cu") (net 2))
@@
   (segment (start 131.2938 98.298) (end 131.2938 97.6123) (width 0.25) (layer "F.Cu") (net 2))
   (segment (start 124.23 101.092) (end 120.65 101.092) (width 0.25) (layer "F.Cu") (net 2))
+  (segment (start 138.684 97.5955) (end 138.684 94.2765) (width 0.25) (layer "F.Cu") (net 2))
   (segment (start 136.7616 99.9494) (end 137.6249 99.0861) (width 0.25) (layer "F.Cu") (net 2))
   (segment (start 123.3581 93.217) (end 123.3581 92.6137) (width 0.25) (layer "F.Cu") (net 2))
   (segment (start 126.1259 100.198) (end 129.032 100.198) (width 0.25) (layer "F.Cu") (net 2))
+  (segment (start 138.413 98.298) (end 138.7845 98.298) (width 0.25) (layer "F.Cu") (net 2))
+  (segment (start 145.739 98.552) (end 144.5621 98.552) (width 0.25) (layer "F.Cu") (net 2))
   (segment (start 136.3555 91.948) (end 136.2475 91.948) (width 0.25) (layer "F.Cu") (net 2))
-  (segment (start 145.739 98.552) (end 144.5621 98.552) (width 0.25) (layer "F.Cu") (net 2))
   (segment (start 131.2938 98.298) (end 133.5035 98.298) (width 0.25) (layer "F.Cu") (net 2))
   (segment (start 120.65 92.116) (end 122.8604 92.116) (width 0.25) (layer "F.Cu") (net 2))
-  (segment (start 137.9815 98.7295) (end 137.9815 98.298) (width 0.25) (layer "F.Cu") (net 2))
   (segment (start 127.6497 89.8748) (end 127.6497 90.8509) (width 0.25) (layer "F.Cu") (net 2))
   (via (at 120.4172 92.3488) (size 0.8) (drill 0.4) (layers "F.Cu" "B.Cu") (net 2))

Commit message: Added v3
Parts:
- added R7: 55, Resistor_SMD:R_0603_1608Metric_Pad0.98x0.95mm_HandSolder, B.Cu at (132.3, 101.9)
- added R8: 5, Resistor_SMD:R_0603_1608Metric_Pad0.98x0.95mm_HandSolder, B.Cu at (130.8, 100.0)
- added R9: 5, Resistor_SMD:R_0603_1608Metric_Pad0.98x0.95mm_HandSolder, B.Cu at (126.5, 99.1)
- D1: footprint LED_THT:LED_D5.0mm-4_RGB -> LED_THT:LED_D5.0mm-4_RGB_Wide_Pins
- Q1: value DMN3300U -> DMN2024U-7
- moved U1 5.84 mm to (136.9, 95.2)
- moved R2 4.89 mm to (131.6, 93.7), turned to 90 degrees
- moved R5 3.61 mm to (139.7, 91.2)
- moved R4 3.59 mm to (139.7, 94.5)
- moved R3 3.42 mm to (139.7, 92.7)
- moved C4 3.24 mm to (131.0, 89.4)
- moved U3 2.96 mm to (136.0, 97.0)
- moved Q1 2.96 mm to (135.9, 93.2)
- moved R1 2.86 mm to (130.0, 93.6), turned to 90 degrees
- moved C2 2.81 mm to (133.1, 95.5)
- moved C3 2.62 mm to (138.9, 97.0)
- moved R6 2.41 mm to (135.6, 89.7)
- moved C5 1.61 mm to (131.1, 90.9), turned to 0 degrees
- moved C1 1.27 mm to (134.4, 99.6)
- moved C6 1.27 mm to (137.9, 99.6)
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Connections:
- D1 pad 1: /LED0 -> Net-(D1-RK)
- D1 pad 2: /LED1 -> Net-(D1-GK)
- D1 pad 4: /LED2 -> Net-(D1-BK)
Routing:
- net GND: track 103.7 -> 141.7 mm, vias 1 -> 0
- net +3.3V: track 30.1 -> 40.9 mm, vias 1 -> 0
- net VBUS: track 25.1 -> 14.4 mm
- net /LED2: track 3.09 -> 10.7 mm
- net Net-(J4-CC2): track 2.24 -> 8.04 mm
- net /BAT_VOLT: track 18.4 -> 12.9 mm
- net /TEMP: track 16.0 -> 11.7 mm
- net Net-(D1-BK): track 0.00 -> 4.27 mm
- net Net-(D1-RK): track 0.00 -> 3.70 mm
- net Net-(J4-CC1): track 2.63 -> 6.15 mm
- net +BATT: track 47.0 -> 50.5 mm, vias 2 -> 1
- net /GATE: track 9.75 -> 7.06 mm
- net /LED0: track 8.46 -> 6.18 mm
- net Net-(D1-GK): track 0.00 -> 2.07 mm
- net /BUTTON: track 30.1 -> 31.5 mm
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Other:
- board size 32.3 x 16.5 mm -> 32.3 x 15.7 mm
