File: heatedGripv3/heatedGripv3.kicad_pcb (KiCad board)
At the start: 2 copper layers, 43.4 x 16.3 mm, 41 parts, among them J1 TEMP, J2 HEAT, J3 BATT, J4 USB_C_Receptacle_PowerOnly_6P, J5 PROG, Q1 DMN2024U-7, Q2 DMN2024U-7, SW1 SW_Push, U1 ATtiny204-SS, U2 MCP73811T-420I-OT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

Commit message: Small tweaks
Parts:
- removed D1: QBL8RGB60D0-2897, LED_THT:LED_D5.0mm-4_RGB_Wide_Pins
- removed JP1: LOGIC_SEL, Jumper:SolderJumper-3_P1.3mm_Open_Pad1.0x1.5mm_NumberLabels
- removed JP2: IN_SEL, Jumper:SolderJumper-3_P1.3mm_Open_Pad1.0x1.5mm_NumberLabels
- removed JP3: OUT_SEL, Jumper:SolderJumper-3_P1.3mm_Open_Pad1.0x1.5mm_NumberLabels
- removed Q2: DMN2024U-7, Package_TO_SOT_SMD:SOT-23
- removed R11: 100, Resistor_SMD:R_0603_1608Metric_Pad0.98x0.95mm_HandSolder
- removed R15: 10k, Resistor_SMD:R_0603_1608Metric_Pad0.98x0.95mm_HandSolder
- added C1: 10u, Capacitor_SMD:C_0603_1608Metric_Pad1.08x0.95mm_HandSolder, B.Cu at (143.8, 96.0)
- added C2: 10u, Capacitor_SMD:C_0603_1608Metric_Pad1.08x0.95mm_HandSolder, B.Cu at (141.0, 93.6)
- added D3: B340, Diode_SMD:D_SMA, B.Cu at (154.2, 90.9)
- added D4: LED_GBAR, LED_THT:LED_D5.0mm-4_RGB_Wide_Pins, F.Cu at (128.8, 96.9)
- R3: value 100k -> 200k
- moved R6 11.3 mm to (139.7, 98.4), turned to 90 degrees
- moved R5 7.50 mm to (142.2, 97.5), turned to 180 degrees
Connections:
- C10 pad 1: /SWITCHING_OUT -> /HEAT_OUT
- D2 pad 1: /SWITCHING_OUT -> /HEAT_OUT
- L1 pad 1: /SWITCHING_POWER -> +BATT
- Q1 pad 3: /SWITCHING_OUT -> /HEAT_OUT
- R14 pad 1: /SWITCHING_OUT -> /HEAT_OUT
- U3 pad 3: +BATT -> Net-(D3-K)
- U4 pad 2: /SWITCHING_POWER -> +BATT
- U4 pad 3: /SWITCHING_EN -> /HEAT_EN
Routing:
- net GND: track 153.0 -> 0.00 mm, vias 4 -> 0
- net /MOSFET_EN: track 32.7 -> 0.00 mm, vias 2 -> 0
- net /BUTTON: track 19.8 -> 0.00 mm
- net +3.3V: track 65.4 -> 47.7 mm, vias 3 -> 0
- net /SWITCHING_POWER: track 14.0 -> 0.00 mm, vias 1 -> 0
- net VBUS: track 13.9 -> 0.00 mm
- net Net-(JP4-A): track 12.6 -> 0.00 mm
- net /SWITCHING_OUT: track 12.2 -> 0.00 mm, vias 1 -> 0
- net /HEAT_OUT: track 3.90 -> 15.5 mm
- net Net-(J4-CC2): track 10.1 -> 0.00 mm, vias 2 -> 0
- net /SWITCHING_EN: track 9.69 -> 0.00 mm, vias 1 -> 0
- net Net-(D3-K): track 0.00 -> 8.45 mm
- net /MOSFET_POWER: track 6.51 -> 0.00 mm
- net Net-(J4-CC1): track 5.90 -> 0.00 mm
- net +BATT: track 28.7 -> 23.1 mm, vias 1 -> 0
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