File: heatedGripv3/heatedGripv3.kicad_sch (KiCad schematic)
At the start: 37 parts, among them J1 TEMP, J2 HEAT, J3 BATT, J4 USB_C_Receptacle_PowerOnly_6P, J5 PROG, Q1 DMN2024U-7, SW1 SW_Push, U1 ATtiny204-SS, U2 MCP73811T-420I-OT, U3 REG710NA-3.3/3K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

Commit message: Added v3
Parts:
- removed C1, C2: 2.2u, Capacitor_SMD:C_0603_1608Metric_Pad1.08x0.95mm_HandSolder, symbol Device:C
- removed C3: 0.22u, Capacitor_SMD:C_0603_1608Metric_Pad1.08x0.95mm_HandSolder, symbol Device:C_Small
- removed U3: REG710NA-3.3/3K, Package_TO_SOT_SMD:TSOT-23-6, symbol velo:REG710NA-3.3/3K
- added JP1: LOGIC_SEL, Jumper:SolderJumper-3_P1.3mm_Open_Pad1.0x1.5mm_NumberLabels, symbol Jumper:SolderJumper_3_Open
- added JP2: IN_SEL, Jumper:SolderJumper-3_P1.3mm_Open_Pad1.0x1.5mm_NumberLabels, symbol Jumper:SolderJumper_3_Open
- added JP3: OUT_SEL, Jumper:SolderJumper-3_P1.3mm_Open_Pad1.0x1.5mm_NumberLabels, symbol Jumper:SolderJumper_3_Open
- added JP4: CHARGER_EN, Jumper:SolderJumper-2_P1.3mm_Open_Pad1.0x1.5mm, symbol Jumper:SolderJumper_2_Open
- added Q2: DMN2024U-7, Package_TO_SOT_SMD:SOT-23, symbol Transistor_FET:DMN3300U
- added R11: 100, Resistor_SMD:R_0603_1608Metric_Pad0.98x0.95mm_HandSolder, symbol Device:R
- added R15: 10k, Resistor_SMD:R_0603_1608Metric_Pad0.98x0.95mm_HandSolder, symbol Device:R
- added U3: MCP1703Ax-330xxTT, Package_TO_SOT_SMD:SOT-23, symbol Regulator_Linear:MCP1703Ax-330xxTT
- C10, C7, C8, C9: footprint (none) -> Capacitor_SMD:C_0603_1608Metric_Pad1.08x0.95mm_HandSolder
- D2: footprint Diode_SMD:D_SMC -> Diode_SMD:D_SMA
- L1: footprint (none) -> Inductor_SMD:L_Bourns_SRP1038C_10.0x10.0mm
- R10, R12, R13, R14: footprint (none) -> Resistor_SMD:R_0603_1608Metric_Pad0.98x0.95mm_HandSolder
- R3: value 100k -> 200k
- U4: footprint SOP-8_PAM2423AECADJR_DIO -> Package_SO:SOIC-8-1EP_3.9x4.9mm_P1.27mm_EP2.29x3mm
Connections:
- net +3.3V: now also U3.2 (VO)
- net +BATT: now also JP2.2 (C), JP4.2 (B), U3.3 (VI); no longer C5.1, L1.1, U2.3 (V_{BAT}), U4.2 (VIN)
- net GND: now also U4.9 (EPAD), R15.1, U3.1 (GND); no longer U4.EPAD
- net HEAT_EN: now also JP1.2 (C); no longer U4.3 (EN)
- net HEAT_OUT: now also JP3.2 (C); no longer C10.1, D2.1 (K), Q1.3 (D), R14.1
- new net: Q2.1 (G), R11.1
- new net: C5.1, JP4.1 (A), U2.3 (V_{BAT})
- new net MOSFET_EN: JP1.3 (B), R11.2, R15.2
- new net MOSFET_OUT: JP3.3 (B), Q2.2 (S)
- new net MOSFET_POWER: JP2.3 (B), Q2.3 (D)
- new net SWITCHING_EN: JP1.1 (A), U4.3 (EN)
- new net SWITCHING_OUT: C10.1, D2.1 (K), JP3.1 (A), Q1.3 (D), R14.1
- new net SWITCHING_POWER: JP2.1 (A), L1.1, U4.2 (VIN)
Other:
- moved on the sheet: C10, C4, C5, C6, C7, C8, C9, D1, D2, J1, J2, J3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

Commit message: Small tweaks
Parts:
- removed D1: QBL8RGB60D0-2897, LED_THT:LED_D5.0mm-4_RGB_Wide_Pins, symbol Device:LED_RGAB
- removed JP1: LOGIC_SEL, Jumper:SolderJumper-3_P1.3mm_Open_Pad1.0x1.5mm_NumberLabels, symbol Jumper:SolderJumper_3_Open
- removed JP2: IN_SEL, Jumper:SolderJumper-3_P1.3mm_Open_Pad1.0x1.5mm_NumberLabels, symbol Jumper:SolderJumper_3_Open
- removed JP3: OUT_SEL, Jumper:SolderJumper-3_P1.3mm_Open_Pad1.0x1.5mm_NumberLabels, symbol Jumper:SolderJumper_3_Open
- removed Q2: DMN2024U-7, Package_TO_SOT_SMD:SOT-23, symbol Transistor_FET:DMN3300U
- removed R11: 100, Resistor_SMD:R_0603_1608Metric_Pad0.98x0.95mm_HandSolder, symbol Device:R
- removed R15: 10k, Resistor_SMD:R_0603_1608Metric_Pad0.98x0.95mm_HandSolder, symbol Device:R
- added C1, C2: 10u, Capacitor_SMD:C_0603_1608Metric_Pad1.08x0.95mm_HandSolder, symbol Device:C
- added D3: B340, Diode_SMD:D_SMA, symbol Diode:B340
- added D4: LED_GBAR, LED_THT:LED_D5.0mm-4_RGB_Wide_Pins, symbol Device:LED_GBAR
Connections:
- net SWITCHING_EN is gone; now on net HEAT_EN: U4.3 (EN)
- net SWITCHING_OUT is gone; now on net HEAT_OUT: C10.1, D2.1 (K), Q1.3 (D), R14.1
- net SWITCHING_POWER is gone; now on net +BATT: L1.1, U4.2 (VIN)
- net +3.3V: now also C2.1, D4.3 (A)
- net +BATT: now also D3.2 (A); no longer U3.3 (VI)
- net GND: now also C1.2, C2.2
- net at R9.2: now also D4.2 (BK)
- net at R7.2: now also D4.4 (RK)
- net at R8.2: now also D4.1 (GK)
- new net: C1.1, D3.1 (K), U3.3 (VI)
